Commit message: slerp added for quaternion interpolation but need to be tuned

File: experiments/models/hook_task/scissors/scissors.urdf (robot description, URDF)
Before this commit: robot donut, 1 links, 0 joints
Links:
- link base_link: geometry collision mesh filename=package://scissors/scissors_vhacd.obj scale=0.002 0.002 0.002; visual mesh filename=package://scissors/scissors.stl scale=0.002 0.002 0.002
