Commit message: hooks fixed

File: experiments/models/hook_task/hook/hook1.urdf (robot description, URDF)
Before this commit: robot hook, 1 links, 0 joints
Links:
- link base_link: geometry collision mesh filename=package://hook/hook1.obj scale=0.1 0.1 0.1; visual mesh filename=package://hook/hook1.stl scale=0.1 0.1 0.1

File: experiments/models/hook_task/slatwall-hook/slatwall_hook.urdf (robot description, URDF)
Before this commit: robot hook, 1 links, 0 joints
Links:
- link base_link: geometry collision mesh filename=package://slatwall-hook/slatwall_vhacd.obj scale=0.002 0.002 0.002; visual mesh filename=package://slatwall-hook/slatwall.stl scale=0.002 0.002 0.002

Commit message: physical sim added for releasing tools, falling and  hooked - manually-assigned release poses

File: experiments/models/hook_task/hook/hook1.urdf (robot description, URDF)
Before this commit: robot hook, 1 links, 0 joints
Links:
- link base_link: geometry collision mesh filename=package://hook/hook1_vhacd.obj scale=0.1 0.1 0.1; visual mesh filename=package://hook/hook1.stl scale=0.1 0.1 0.1

File: experiments/models/hook_task/scissors/scissors.urdf (robot description, URDF)
Before this commit: robot donut, 1 links, 0 joints
Links:
- link base_link: geometry collision mesh filename=package://scissors/scissors_vhacd.obj scale=0.0015 0.0015 0.0015; visual mesh filename=package://scissors/scissors.stl scale=0.0015 0.0015 0.0015

File: experiments/models/hook_task/tape/tape.urdf (robot description, URDF)
Before this commit: robot donut, 1 links, 0 joints
Links:
- link base_link: geometry collision mesh filename=package://tape/tape_vhacd.obj scale=1.2 1.2 1.2; visual mesh filename=package://tape/tape.stl scale=1.2 1.2 1.2
